Commit message: 2021年 03月 13日 星期六 19:27:14 CST

File: demo/ur3_joint_limited_robot.urdf (robot description, URDF)
Before this commit: robot ur3, 11 links, 10 joints
Links:
- link base_link: geometry collision mesh filename=package://ur3_pybullet_data/meshes/ur3/collision/base.stl; visual mesh filename=package://ur3_pybullet_data/meshes/ur3/visual/base.dae
- link forearm_link: geometry collision mesh filename=package://ur3_pybullet_data/meshes/ur3/collision/forearm.stl; visual mesh filename=package://ur3_pybullet_data/meshes/ur3/visual/forearm.dae
- link shoulder_link: geometry collision mesh filename=package://ur3_pybullet_data/meshes/ur3/collision/shoulder.s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; visual mesh filename=package://ur3_pybullet_data/meshes/ur3/visual/shoulder.dae
- link upper_arm_link: geometry collision mesh filename=package://ur3_pybullet_data/meshes/ur3/collision/upperarm.s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; visual mesh filename=package://ur3_pybullet_data/meshes/ur3/visual/upperarm.dae
- link wrist_1_link: geometry collision mesh filename=package://ur3_pybullet_data/meshes/ur3/collision/wrist1.stl; visual mesh filename=package://ur3_pybullet_data/meshes/ur3/visual/wrist1.dae
- link wrist_2_link: geometry collision mesh filename=package://ur3_pybullet_data/meshes/ur3/collision/wrist2.stl; visual mesh filename=package://ur3_pybullet_data/meshes/ur3/visual/wrist2.dae
- link wrist_3_link: geometry collision mesh filename=package://ur3_pybullet_data/meshes/ur3/collision/wrist3.stl; visual mesh filename=package://ur3_pybullet_data/meshes/ur3/visual/wrist3.dae

File: demo/ur3_visual_grabbing_with_rg2.urdf (robot description, URDF)
Before this commit: robot ur3_visual_grabbing, 26 links, 25 joints
Links:
- link base_link: geometry collision mesh filename=package://ur3_pybullet_data/meshes/ur3/collision/base.stl; visual mesh filename=package://ur3_pybullet_data/meshes/ur3/visual/base.dae
- link forearm_link: geometry collision mesh filename=package://ur3_pybullet_data/meshes/ur3/collision/forearm.stl; visual mesh filename=package://ur3_pybullet_data/meshes/ur3/visual/forearm.dae
- link ft300_mounting_plate: geometry collision mesh filename=package://ur3_pybullet_data/meshes/robotiq_ft_sensor/collis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; visual mesh filename=package://ur3_pybullet_data/meshes/robotiq_ft_sensor/visual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
- link ft300_sensor: geometry collision mesh filename=package://ur3_pybullet_data/meshes/robotiq_ft_sensor/collis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; visual mesh filename=package://ur3_pybullet_data/meshes/robotiq_ft_sensor/visual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
- link gripper_base_link: geometry collision mesh filename=package://ur3_pybullet_data/meshes/onrobot_rg2/collision/gr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; visual mesh filename=package://ur3_pybullet_data/meshes/onrobot_rg2/visual/gripp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
- link gripper_finger1_finger_link: geometry collision mesh filename=package://ur3_pybullet_data/meshes/onrobot_rg2/collision/gr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; visual mesh filename=package://ur3_pybullet_data/meshes/onrobot_rg2/visual/gripp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
- link gripper_finger1_finger_tip_link: geometry collision mesh filename=package://ur3_pybullet_data/meshes/onrobot_rg2/collision/gr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; visual mesh filename=package://ur3_pybullet_data/meshes/onrobot_rg2/visual/gripp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
- link gripper_finger1_inner_knuckle_link: geometry collision mesh filename=package://ur3_pybullet_data/meshes/onrobot_rg2/collision/gr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; visual mesh filename=package://ur3_pybullet_data/meshes/onrobot_rg2/visual/gripp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
- link gripper_finger2_finger_link: geometry collision mesh filename=package://ur3_pybullet_data/meshes/onrobot_rg2/collision/gr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; visual mesh filename=package://ur3_pybullet_data/meshes/onrobot_rg2/visual/gripp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
- link gripper_finger2_finger_tip_link: geometry collision mesh filename=package://ur3_pybullet_data/meshes/onrobot_rg2/collision/gr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; visual mesh filename=package://ur3_pybullet_data/meshes/onrobot_rg2/visual/gripp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
- link gripper_finger2_inner_knuckle_link: geometry collision mesh filename=package://ur3_pybullet_data/meshes/onrobot_rg2/collision/gr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; visual mesh filename=package://ur3_pybullet_data/meshes/onrobot_rg2/visual/gripp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
- link kinect2_base_link: geometry collision mesh filename=package://ur3_pybullet_data/meshes/kinect_v2/kinect2.STL; visual mesh filename=package://ur3_pybullet_data/meshes/kinect_v2/kinect2.STL
- link shoulder_link: geometry collision mesh filename=package://ur3_pybullet_data/meshes/ur3/collision/shoulder.s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; visual mesh filename=package://ur3_pybullet_data/meshes/ur3/visual/shoulder.dae
- link upper_arm_link: geometry collision mesh filename=package://ur3_pybullet_data/meshes/ur3/collision/upperarm.s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; visual mesh filename=package://ur3_pybullet_data/meshes/ur3/visual/upperarm.dae
- link wrist_1_link: geometry collision mesh filename=package://ur3_pybullet_data/meshes/ur3/collision/wrist1.stl; visual mesh filename=package://ur3_pybullet_data/meshes/ur3/visual/wrist1.dae
- link wrist_2_link: geometry collision mesh filename=package://ur3_pybullet_data/meshes/ur3/collision/wrist2.stl; visual mesh filename=package://ur3_pybullet_data/meshes/ur3/visual/wrist2.dae
- link wrist_3_link: geometry collision mesh filename=package://ur3_pybullet_data/meshes/ur3/collision/wrist3.stl; visual mesh filename=package://ur3_pybullet_data/meshes/ur3/visual/wrist3.dae

File: kinect_v2.urdf (robot description, URDF)
Before this commit: robot kinect_v2, 6 links, 5 joints
Links:
- link kinect2_base_link: geometry collision mesh filename=package://ur3_pybullet_data/meshes/kinect_v2/kinect2.STL; visual mesh filename=package://ur3_pybullet_data/meshes/kinect_v2/kinect2.STL

File: object_demo.urdf (robot description, URDF)
Before this commit: robot airplane, 1 links, 0 joints
Links:
- link base: geometry collision mesh filename=package://ur3_pybullet_data/meshes/objects/828d1b43814fc98c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

File: onrobot_rg2.urdf (robot description, URDF)
Before this commit: robot onrobot_rg2, 9 links, 8 joints
Links:
- link gripper_base_link: geometry collision mesh filename=package://ur3_pybullet_data/meshes/onrobot_rg2/collision/gr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; visual mesh filename=package://ur3_pybullet_data/meshes/onrobot_rg2/visual/gripp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
- link gripper_finger1_finger_link: geometry collision mesh filename=package://ur3_pybullet_data/meshes/onrobot_rg2/collision/gr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; visual mesh filename=package://ur3_pybullet_data/meshes/onrobot_rg2/visual/gripp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
- link gripper_finger1_finger_tip_link: geometry collision mesh filename=package://ur3_pybullet_data/meshes/onrobot_rg2/collision/gr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; visual mesh filename=package://ur3_pybullet_data/meshes/onrobot_rg2/visual/gripp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
- link gripper_finger1_inner_knuckle_link: geometry collision mesh filename=package://ur3_pybullet_data/meshes/onrobot_rg2/collision/gr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; visual mesh filename=package://ur3_pybullet_data/meshes/onrobot_rg2/visual/gripp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
- link gripper_finger2_finger_link: geometry collision mesh filename=package://ur3_pybullet_data/meshes/onrobot_rg2/collision/gr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; visual mesh filename=package://ur3_pybullet_data/meshes/onrobot_rg2/visual/gripp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
- link gripper_finger2_finger_tip_link: geometry collision mesh filename=package://ur3_pybullet_data/meshes/onrobot_rg2/collision/gr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; visual mesh filename=package://ur3_pybullet_data/meshes/onrobot_rg2/visual/gripp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
- link gripper_finger2_inner_knuckle_link: geometry collision mesh filename=package://ur3_pybullet_data/meshes/onrobot_rg2/collision/gr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; visual mesh filename=package://ur3_pybullet_data/meshes/onrobot_rg2/visual/gripp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

File: ur3_visual_grabbing_with_rg2.urdf (robot description, URDF)
Before this commit: robot ur3_visual_grabbing, 20 links, 19 joints
Links:
- link base_link: geometry collision mesh filename=package://ur3_pybullet_data/meshes/ur3/collision/base.stl; visual mesh filename=package://ur3_pybullet_data/meshes/ur3/visual/base.dae
- link forearm_link: geometry collision mesh filename=package://ur3_pybullet_data/meshes/ur3/collision/forearm.stl; visual mesh filename=package://ur3_pybullet_data/meshes/ur3/visual/forearm.dae
- link ft300_mounting_plate: geometry collision mesh filename=package://ur3_pybullet_data/meshes/robotiq_ft_sensor/collis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; visual mesh filename=package://ur3_pybullet_data/meshes/robotiq_ft_sensor/visual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
- link ft300_sensor: geometry collision mesh filename=package://ur3_pybullet_data/meshes/robotiq_ft_sensor/collis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; visual mesh filename=package://ur3_pybullet_data/meshes/robotiq_ft_sensor/visual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
- link gripper_base_link: geometry collision mesh filename=package://ur3_pybullet_data/meshes/onrobot_rg2/collision/gr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; visual mesh filename=package://ur3_pybullet_data/meshes/onrobot_rg2/visual/gripp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
- link gripper_finger1_finger_link: geometry collision mesh filename=package://ur3_pybullet_data/meshes/onrobot_rg2/collision/gr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; visual mesh filename=package://ur3_pybullet_data/meshes/onrobot_rg2/visual/gripp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
- link gripper_finger1_finger_tip_link: geometry collision mesh filename=package://ur3_pybullet_data/meshes/onrobot_rg2/collision/gr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; visual mesh filename=package://ur3_pybullet_data/meshes/onrobot_rg2/visual/gripp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
- link gripper_finger1_inner_knuckle_link: geometry collision mesh filename=package://ur3_pybullet_data/meshes/onrobot_rg2/collision/gr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; visual mesh filename=package://ur3_pybullet_data/meshes/onrobot_rg2/visual/gripp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
- link gripper_finger2_finger_link: geometry collision mesh filename=package://ur3_pybullet_data/meshes/onrobot_rg2/collision/gr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; visual mesh filename=package://ur3_pybullet_data/meshes/onrobot_rg2/visual/gripp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
- link gripper_finger2_finger_tip_link: geometry collision mesh filename=package://ur3_pybullet_data/meshes/onrobot_rg2/collision/gr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; visual mesh filename=package://ur3_pybullet_data/meshes/onrobot_rg2/visual/gripp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
- link gripper_finger2_inner_knuckle_link: geometry collision mesh filename=package://ur3_pybullet_data/meshes/onrobot_rg2/collision/gr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; visual mesh filename=package://ur3_pybullet_data/meshes/onrobot_rg2/visual/gripp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
- link shoulder_link: geometry collision mesh filename=package://ur3_pybullet_data/meshes/ur3/collision/shoulder.s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; visual mesh filename=package://ur3_pybullet_data/meshes/ur3/visual/shoulder.dae
- link upper_arm_link: geometry collision mesh filename=package://ur3_pybullet_data/meshes/ur3/collision/upperarm.s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; visual mesh filename=package://ur3_pybullet_data/meshes/ur3/visual/upperarm.dae
- link wrist_1_link: geometry collision mesh filename=package://ur3_pybullet_data/meshes/ur3/collision/wrist1.stl; visual mesh filename=package://ur3_pybullet_data/meshes/ur3/visual/wrist1.dae
- link wrist_2_link: geometry collision mesh filename=package://ur3_pybullet_data/meshes/ur3/collision/wrist2.stl; visual mesh filename=package://ur3_pybullet_data/meshes/ur3/visual/wrist2.dae
- link wrist_3_link: geometry collision mesh filename=package://ur3_pybullet_data/meshes/ur3/collision/wrist3.stl; visual mesh filename=package://ur3_pybullet_data/meshes/ur3/visual/wrist3.dae
